File: schematic/round/round-sensor.kicad_pcb (KiCad board)
At the start: 2 copper layers, 30 x 30 mm, 28 parts, among them P1 BUS, P2 BUS, P3 SWD, P4 PA0, P5 PA1, P6 PA3, P7 PA10, P8 V+, P9 V-, Q1 Q_NMOS_GSD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

Commit message: PCB improved
Parts:
- added Q3: Q_NMOS_GSD, TO_SOT_Packages_SMD:SOT-23, B.Cu at (6.27, -6.62)
- added R7: 10k, Resistors_SMD:R_0805, B.Cu at (5.67, -9.91)
- added R8: R_load, Resistors_SMD:R_0805, B.Cu at (10.1, -3.67)
- U3: value RGB-LED -> RGB
- moved P7 25.0 mm to (13.2, -0.05)
- moved P5 24.2 mm to (-11.5, 3.44)
- moved C1 2.99 mm to (-5.61, -10.0), turned to 0 degrees
- moved U1 1.87 mm to (-5.14, -6.41)
- moved R5 1.63 mm to (9.59, -4.68)
- moved D1 1.52 mm to (1.27, -7.21)
- moved C4 1.40 mm to (6.01, 5.69), turned to 180 degrees
- moved C3 1.35 mm to (-5.47, -7.34)
- moved R4 0.83 mm to (2.50, 6.57), turned to 270 degrees
- moved R1 0.72 mm to (-5.54, 3.39), turned to 90 degrees
- moved R6 0.64 mm to (6.26, -9.99)
- moved C2 0.60 mm to (-8.72, -7.06)
- moved R3 0.49 mm to (-5.94, 7.86)
- moved Q2 0.46 mm to (6.48, -6.77)
- moved R2 0.41 mm to (-6.11, 5.92)
Connections:
- P7 pad 1: PA10 -> Net-(P7-Pad1)
Routing:
- net VCC: track 56.2 -> 86.2 mm
- net GND: track 31.8 -> 22.2 mm, vias 2 -> 4
- net red: track 16.2 -> 9.59 mm, vias 3 -> 1
- net Net-(Q3-Pad3): track 0.00 -> 6.26 mm
- net PA10: track 11.7 -> 17.8 mm, vias 1 -> 2
- net Net-(P7-Pad1): track 0.00 -> 5.22 mm
- net PA1: track 13.4 -> 18.3 mm, vias 2 -> 3
- net green: track 14.5 -> 9.87 mm, vias 3 -> 1
- net Net-(C4-Pad2): track 7.67 -> 9.74 mm
- net Bus: track 28.4 -> 29.9 mm, vias 1 -> 2
- net Net-(D1-Pad1): track 4.11 -> 5.61 mm
- net +3V3: track 28.1 -> 26.7 mm, vias 1 -> 2
- net IR_out: track 20.6 -> 21.5 mm
- net Vibro: track 7.55 -> 7.03 mm
- net Net-(R3-Pad1): track 2.12 -> 2.63 mm
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- added copper zone on F.Cu, net VCC
Other:
- net class Default: trace_width 0.6 -> 0.35
- board text added: "Smart sensor rev. R1.0"
